File: Wordclock.kicad_sch (KiCad schematic)
At the start: 224 parts, among them J1 Barrel_Jack, J2 Conn_01x03_Male, J3 Conn_01x03_Male, J4 Screw_Terminal_01x02

Commit message: - first final version
Parts:
- added J5: Screw_Terminal_01x02, TerminalBlock:TerminalBlock_bornier-2_P5.08mm, symbol Connector:Screw_Terminal_01x02
Connections:
- net +5V: now also J5.2 (Pin_2)
- net GND: now also J5.1 (Pin_1)
Changed lines of the file:
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@@
+    (pin "2")
+  )
+  (symbol (lib_id "Connector:Screw_Terminal_01x02") (at 214.63 223.52 180) (unit 1)
+    (in_bom yes) (on_board yes) (fields_autoplaced)
+    (property "Reference" "J5" (id 0) (at 214.63 216.0102 0))
+    (property "Value" "Screw_Terminal_01x02" (id 1) (at 214.63 218.5471 0))
+    (property "Footprint" "TerminalBlock:TerminalBlock_bornier-2_P5.08mm" (id 2) (at 214.63 223.52 0)
+      (effects (font (size 1.27 1.27)) hide)
+    )
+    (property "Datasheet" "~" (id 3) (at 214.63 223.52 0)
+      (effects (font (size 1.27 1.27)) hide)
+    )
+    (pin "1")
     (pin "2")
   )
@@
     (pin "2")
   )
+  (symbol (lib_id "power:GND") (at 219.71 223.52 90) (unit 1)
+    (in_bom yes) (on_board yes) (fields_autoplaced)
+    (property "Reference" "#PWR0108" (id 0) (at 226.06 223.52 0)
+      (effects (font (size 1.27 1.27)) hide)
+    )
+    (property "Value" "GND" (id 1) (at 222.885 223.9538 90)
+      (effects (font (size 1.27 1.27)) (justify right))
+    )
+    (property "Footprint" "" (id 2) (at 219.71 223.52 0)
+      (effects (font (size 1.27 1.27)) hide)
+    )
+    (property "Datasheet" "" (id 3) (at 219.71 223.52 0)
+      (effects (font (size 1.27 1.27)) hide)
+    )
+    (pin "1")
+  )
   (symbol (lib_id "power:GND") (at 25.4 166.37 270) (unit 1)
     (in_bom yes) (on_board yes) (fields_autoplaced)
@@
     )
     (property "Datasheet" "" (id 3) (at 25.4 130.81 0)
+      (effects (font (size 1.27 1.27)) hide)
+    )
+    (pin "1")
+  )
+  (symbol (lib_id "power:+5V") (at 219.71 220.98 270) (unit 1)
+    (in_bom yes) (on_board yes) (fields_autoplaced)
+    (property "Reference" "#PWR0107" (id 0) (at 215.9 220.98 0)
+      (effects (font (size 1.27 1.27)) hide)
+    )
+    (property "Value" "+5V" (id 1) (at 222.885 221.4138 90)
+      (effects (font (size 1.27 1.27)) (justify left))
+    )
+    (property "Footprint" "" (id 2) (at 219.71 220.98 0)
+      (effects (font (size 1.27 1.27)) hide)
+    )
+    (property "Datasheet" "" (id 3) (at 219.71 220.98 0)
       (effects (font (size 1.27 1.27)) hide)
     )
@@
       (reference "#PWR0106") (unit 1) (value "+5V") (footprint "")
     )
+    (path "/a86e8a6a-4a69-44ee-b851-2e958dc4871a"
+      (reference "#PWR0107") (unit 1) (value "+5V") (footprint "")
+    )
+    (path "/9e16a819-e393-4105-923b-2a2246068467"
+      (reference "#PWR0108") (unit 1) (value "GND") (footprint "")
+    )
     (path "/02908c32-dce5-4198-9a37-57f9d737afb4"
       (reference "C1") (unit 1) (value "C") (footprint "Capacitor_SMD:C_0805_2012Metric_Pad1.18x1.45mm_HandSolder")
@@
       (reference "J4") (unit 1) (value "Screw_Terminal_01x02") (footprint "TerminalBlock:TerminalBlock_bornier-2_P5.08mm")
     )
-  )
+    (path "/75290e04-49c5-4682-9b06-762a5c131876"
+      (reference "J5") (unit 1) (value "Screw_Terminal_01x02") (footprint "TerminalBlock:TerminalBlock_bornier-2_P5.08mm")
+    )
+  )
